Commit message: 碰撞模型更加符合实际

File: urdf/dog_v2_2_4.urdf (robot description, URDF)
Before this commit: robot dog_v2_go2_aligned, 17 links, 16 joints
Links:
- link FL_thigh: geometry collision box size=0.2054269677 0.05 0.025; visual mesh filename=../meshes/LF_HipF_link.STL
- link FR_thigh: geometry collision box size=0.2054269677 0.05 0.025; visual mesh filename=../meshes/RF_HipF_link.STL
- link RL_thigh: geometry collision box size=0.2054269677 0.05 0.025; visual mesh filename=../meshes/LR_HipF_link.STL
- link RR_thigh: geometry collision box size=0.2054269677 0.05 0.025; visual mesh filename=../meshes/RR_HipF_link.STL
- link base: geometry collision box size=0.52 0.16 0.12; visual mesh filename=../meshes/base_link.STL

Commit message: 优化添加一个头,防止因为头导致重置并且身子重置应该保留,优化hip还有thigh之间碰撞体

File: urdf/dog_v2_2_4.urdf (robot description, URDF)
Before this commit: robot dog_v2_go2_aligned, 17 links, 16 joints
Links:
- added link Head_upper, mass 0.001; collision box size=0.12 0.12 0.12
- link FL_thigh: geometry collision box size=0.1404269677 0.05 0.025; visual mesh filename=../meshes/LF_HipF_link.STL
- link FR_thigh: geometry collision box size=0.1404269677 0.05 0.025; visual mesh filename=../meshes/RF_HipF_link.STL
- link RL_thigh: geometry collision box size=0.1404269677 0.05 0.025; visual mesh filename=../meshes/LR_HipF_link.STL
- link RR_thigh: geometry collision box size=0.1404269677 0.05 0.025; visual mesh filename=../meshes/RR_HipF_link.STL
- link base: geometry collision box size=0.40 0.16 0.12; visual mesh filename=../meshes/base_link.STL
Joints:
- added joint Head_upper_joint: type fixed, parent base, child Head_upper, origin xyz=0.225 0 0.01 rpy=0 0 0, axis 0 0 0

Commit message: 优化碰撞模型防止自碰撞calf和thigh

File: urdf/dog_v2_2_4.urdf (robot description, URDF)
Before this commit: robot dog_v2_go2_aligned, 18 links, 17 joints
Links:
- link FL_thigh: geometry collision box size=0.1104269677 0.05 0.025; visual mesh filename=../meshes/LF_HipF_link.STL
- link FR_thigh: geometry collision box size=0.1104269677 0.05 0.025; visual mesh filename=../meshes/RF_HipF_link.STL
- link RL_thigh: geometry collision box size=0.1104269677 0.05 0.025; visual mesh filename=../meshes/LR_HipF_link.STL
- link RR_thigh: geometry collision box size=0.1104269677 0.05 0.025; visual mesh filename=../meshes/RR_HipF_link.STL

Commit message: 注释不需要的headerlink

File: urdf/dog_v2_2_4.urdf (robot description, URDF)
Before this commit: robot dog_v2_go2_aligned, 18 links, 17 joints
Links:
- removed link Head_upper
Joints:
- removed joint Head_upper_joint

Commit message: fix(urdf): 更新四足机器人腿部关节限位范围
调整了FL/FR/RL/RR大腿关节的运动上限/下限值，扩大单侧大腿的活动角度范围

File: urdf/dog_v2_2_4.urdf (robot description, URDF)
Before this commit: robot dog_v2_go2_aligned, 17 links, 16 joints
Joints:
- joint FL_thigh_joint: limit lower=-1.2217658 upper=0.8726683 effort=17 velocity=50 -> lower=-1.2217658 upper=1.5 effort=17 velocity=50
- joint FR_thigh_joint: limit lower=-0.8726999 upper=1.2217342 effort=17 velocity=50 -> lower=-1.5 upper=1.2217342 effort=17 velocity=50
- joint RL_thigh_joint: limit lower=-1.2217305 upper=0.8726683 effort=17 velocity=50 -> lower=-1.2217305 upper=1.5 effort=17 velocity=50
- joint RR_thigh_joint: limit lower=-0.8726999 upper=1.2217305 effort=17 velocity=50 -> lower=-1.5 upper=1.2217305 effort=17 velocity=50

Commit message: 加入回去那个前面头部内容

File: urdf/dog_v2_2_4.urdf (robot description, URDF)
Before this commit: robot dog_v2_go2_aligned, 17 links, 16 joints
Links:
- added link Head_upper, mass 0.001; collision box size=0.12 0.12 0.12
Joints:
- added joint Head_upper_joint: type fixed, parent base, child Head_upper, origin xyz=0.225 0 0.01 rpy=0 0 0, axis 0 0 0
