Commit message: 新增换名字的urdf并且使用mesh作为碰撞体

File: urdf/backup/dog_v2_old_naming.urdf (robot description, URDF)
Before this commit: robot dog_v2_go2_aligned, 17 links, 16 joints
Links:
- removed link FL_calf
- removed link FL_foot
- removed link FL_hip
- removed link FL_thigh
- removed link FR_calf
- removed link FR_foot
- removed link FR_hip
- removed link FR_thigh
- removed link RL_calf
- removed link RL_foot
- removed link RL_hip
- removed link RL_thigh
- removed link RR_calf
- removed link RR_foot
- removed link RR_hip
- removed link RR_thigh
- removed link base
- added link LF_Foot_link, mass 0.038528; collision mesh filename=../meshes/LF_Foot_link.STL; visual mesh filename=../meshes/LF_Foot_link.STL
- added link LF_HipA_link, mass 0.452382; collision mesh filename=../meshes/LF_HipA_link.STL; visual mesh filename=../meshes/LF_HipA_link.STL
- added link LF_HipF_link, mass 0.779164; collision mesh filename=../meshes/LF_HipF_link.STL; visual mesh filename=../meshes/LF_HipF_link.STL
- added link LF_Knee_link, mass 0.121558; collision mesh filename=../meshes/LF_Knee_link.STL; visual mesh filename=../meshes/LF_Knee_link.STL
- added link LR_Foot_link, mass 0.038528; collision mesh filename=../meshes/LR_Foot_link.STL; visual mesh filename=../meshes/LR_Foot_link.STL
- added link LR_HipA_link, mass 0.452382; collision mesh filename=../meshes/LR_HipA_link.STL; visual mesh filename=../meshes/LR_HipA_link.STL
- added link LR_HipF_link, mass 0.779164; collision mesh filename=../meshes/LR_HipF_link.STL; visual mesh filename=../meshes/LR_HipF_link.STL
- added link LR_Knee_link, mass 0.121558; collision mesh filename=../meshes/LR_Knee_link.STL; visual mesh filename=../meshes/LR_Knee_link.STL
- added link RF_Foot_link, mass 0.038528; collision mesh filename=../meshes/RF_Foot_link.STL; visual mesh filename=../meshes/RF_Foot_link.STL
- added link RF_HipA_link, mass 0.452382; collision mesh filename=../meshes/RF_HipA_link.STL; visual mesh filename=../meshes/RF_HipA_link.STL
- added link RF_HipF_link, mass 0.779164; collision mesh filename=../meshes/RF_HipF_link.STL; visual mesh filename=../meshes/RF_HipF_link.STL
- added link RF_Knee_link, mass 0.121558; collision mesh filename=../meshes/RF_Knee_link.STL; visual mesh filename=../meshes/RF_Knee_link.STL
- added link RR_Foot_link, mass 0.038528; collision mesh filename=../meshes/RR_Foot_link.STL; visual mesh filename=../meshes/RR_Foot_link.STL
- added link RR_HipA_link, mass 0.452382; collision mesh filename=../meshes/RR_HipA_link.STL; visual mesh filename=../meshes/RR_HipA_link.STL
- added link RR_HipF_link, mass 0.779164; collision mesh filename=../meshes/RR_HipF_link.STL; visual mesh filename=../meshes/RR_HipF_link.STL
- added link RR_Knee_link, mass 0.121558; collision mesh filename=../meshes/RR_Knee_link.STL; visual mesh filename=../meshes/RR_Knee_link.STL
- added link base_link, mass 5.276437; collision mesh filename=../meshes/base_link.STL; visual mesh filename=../meshes/base_link.STL
Joints:
- removed joint FL_calf_joint
- removed joint FL_foot_joint
- removed joint FL_hip_joint
- removed joint FL_thigh_joint
- removed joint FR_calf_joint
- removed joint FR_foot_joint
- removed joint FR_hip_joint
- removed joint FR_thigh_joint
- removed joint RL_calf_joint
- removed joint RL_foot_joint
- removed joint RL_hip_joint
- removed joint RL_thigh_joint
- removed joint RR_calf_joint
- removed joint RR_foot_joint
- removed joint RR_hip_joint
- removed joint RR_thigh_joint
- added joint LF_Foot_joint: type fixed, parent LF_Knee_link, child LF_Foot_link, origin xyz=-0.110125305788291 -0.190742624824423 0.0164999999999972 rpy=1.5707963267949 0 3.14159265358979, axis 0 0 0
- added joint LF_HipA_joint: type revolute, parent base_link, child LF_HipA_link, origin xyz=0.16 0.0674994572689366 0.0630000490222146 rpy=1.5707963267949 0 1.5707963267949, axis 0 0 1, limit lower=-0.7853982 upper=0.7853982 effort=17 velocity=50
- added joint LF_HipF_joint: type revolute, parent LF_HipA_link, child LF_HipF_link, origin xyz=0.018001 0 0.048001 rpy=0 1.5708 0, axis 0 0 1, limit lower=-1.2217658 upper=0.8726683 effort=17 velocity=50
- added joint LF_Knee_joint: type revolute, parent LF_HipF_link, child LF_Knee_link, origin xyz=0.170743431939306 -0.122257424197791 0.0500000000000068 rpy=0 0 0, axis 0 0 1, limit lower=-1.2217299 upper=0.69813 effort=25 velocity=50
- added joint LR_Foot_joint: type fixed, parent LR_Knee_link, child LR_Foot_link, origin xyz=-0.110125305788291 -0.190742624824423 0.0164999999999997 rpy=1.5707963267949 0 -3.14159265358979, axis 0 0 0
- added joint LR_HipA_joint: type revolute, parent base_link, child LR_HipA_link, origin xyz=-0.16 0.0674994572689466 0.0629999509777641 rpy=1.5707963267949 0 -1.5707963267949, axis 0 0 1, limit lower=-0.7853982 upper=0.7853982 effort=17 velocity=50
- added joint LR_HipF_joint: type revolute, parent LR_HipA_link, child LR_HipF_link, origin xyz=-0.018001 0 0.048001 rpy=0 -1.5708 0, axis 0 0 1, limit lower=-1.2217305 upper=0.8726683 effort=17 velocity=50
- added joint LR_Knee_joint: type revolute, parent LR_HipF_link, child LR_Knee_link, origin xyz=0.17074234647718 -0.122257326153361 0.050000000000001 rpy=0 0 0, axis 0 0 1, limit lower=-1.2217299 upper=0.69813 effort=25 velocity=50
- added joint RF_Foot_joint: type fixed, parent RF_Knee_link, child RF_Foot_link, origin xyz=0.110125305788291 -0.190742624824423 0.0165000000000002 rpy=-1.5707963267949 0 0, axis 0 0 0
- added joint RF_HipA_joint: type revolute, parent base_link, child RF_HipA_link, origin xyz=0.16 -0.0674994572689349 0.0629999509777826 rpy=1.5707963267949 0 1.5707963267949, axis 0 0 1, limit lower=-0.7853982 upper=0.7853982 effort=17 velocity=50
- added joint RF_HipF_joint: type revolute, parent RF_HipA_link, child RF_HipF_link, origin xyz=-0.018001 0 0.048001 rpy=0 -1.5708 0, axis 0 0 1, limit lower=-0.8726999 upper=1.2217342 effort=17 velocity=50
- added joint RF_Knee_joint: type revolute, parent RF_HipF_link, child RF_Knee_link, origin xyz=-0.17074 -0.12226 0.05 rpy=0 0 0, axis 0 0 1, limit lower=-0.6981312 upper=1.2217287 effort=25 velocity=50
- added joint RR_Foot_joint: type fixed, parent RR_Knee_link, child RR_Foot_link, origin xyz=0.11013 -0.19074 0.0165 rpy=-1.5708 0 0, axis 0 0 0
- added joint RR_HipA_joint: type revolute, parent base_link, child RR_HipA_link, origin xyz=-0.16 -0.0674994572689364 0.0630000490222165 rpy=1.5707963267949 0 -1.5707963267949, axis 0 0 1, limit lower=-0.7853982 upper=0.7853982 effort=17 velocity=50
- added joint RR_HipF_joint: type revolute, parent RR_HipA_link, child RR_HipF_link, origin xyz=0.018001 0 0.048001 rpy=0 1.5708 0, axis 0 0 1, limit lower=-0.8726999 upper=1.2217305 effort=17 velocity=50
- added joint RR_Knee_joint: type revolute, parent RR_HipF_link, child RR_Knee_link, origin xyz=-0.170742346477182 -0.122257424197793 0.050000000000007 rpy=0 0 0, axis 0 0 1, limit lower=-0.6981312 upper=1.2217287 effort=25 velocity=50
